File: DC_Board/DC_Board.kicad_pcb (KiCad board)
At the start: 2 copper layers, 169 x 160 mm, 43 parts, among them J1 0039281243, J10 15-24-4449, J11 Conn_01x03_Male, J12 Conn_01x02_Male, J13 Conn_01x02_Male, J2 0039281243, J3 26-01-3115, J4 26-01-3115, J5 26-01-3115, J6 26-01-3115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

Commit message: Brand new AC and DC boards
Parts:
- removed D1: 1N4001, Diode_THT:D_DO-41_SOD81_P10.16mm_Horizontal
- removed J13: Conn_01x02_Male, Connector_Molex:Molex_KK-254_AE-6410-02A_1x02_P2.54mm_Vertical
- removed K1: EC2-12NU, Relay_12:RELAY_EC2-5NU
- removed R3, R4: R, Resistor_THT:R_Axial_Power_L38.0mm_W9.0mm_P45.72mm
- removed the REF** at (274.4, 186.4)
- removed the REF** at (259.0, 105.9)
- added REF**: MountingHole_4mm, MountingHole:MountingHole_4mm, F.Cu at (170.0, 150.0)
- added REF**: MountingHole_4mm, MountingHole:MountingHole_4mm, F.Cu at (170.0, 140.0)
- added REF**: OSHW-Logo2_9.8x8mm_SilkScreen, Symbol:OSHW-Logo2_9.8x8mm_SilkScreen, F.Cu at (315.0, 219.3)
- added REF**: MountingHole_4mm, MountingHole:MountingHole_4mm, F.Cu at (297.3, 179.1)
- added REF**: MountingHole_4mm, MountingHole:MountingHole_4mm, F.Cu at (259.3, 78.4)
- added TP1: TestPoint_2Pole, Connector_PinHeader_2.54mm:PinHeader_2x01_P2.54mm_Vertical, F.Cu at (205.0, 203.8)
- J1: footprint Connector_Molex:Molex_Mini-Fit_Jr_5566-24A_2x12_P4.20mm_Vertical -> Connector_Molex:Molex_Mini-Fit_Jr_5566-24A2_2x12_P4.20mm_Vertical
- J10, J7, J8, J9: footprint Connector_TE-Connectivity:TE_MATE-N-LOK_350211-1_1x04_P5.08mm_Vertical -> Molex_Right_Angle:641737-1
- J12: footprint Connector_Molex:Molex_KK-254_AE-6410-02A_1x02_P2.54mm_Vertical -> Connector_Molex:Molex_KK-396_A-41791-0002_1x02_P3.96mm_Vertical
- TH1: footprint Connector_PinHeader_2.54mm:PinHeader_1x02_P2.54mm_Vertical -> Resistor_THT:R_Axial_DIN0309_L9.0mm_D3.2mm_P15.24mm_Horizontal
- moved J12 121.9 mm to (169.2, 90.1), turned to 90 degrees
- moved J10 87.7 mm to (186.1, 99.5), turned to 180 degrees
- moved G*** 81.7 mm to (307.7, 91.7), turned to 0 degrees
- moved G*** 80.4 mm to (293.5, 93.1), turned to 90 degrees
- moved J7 77.7 mm to (268.4, 99.7), turned to 180 degrees
- moved D2 50.3 mm to (191.6, 220.2)
- moved R7 36.6 mm to (200.6, 183.3), turned to 180 degrees
- moved J9 34.8 mm to (213.6, 99.5), turned to 180 degrees
- moved J1 30.9 mm to (313.2, 122.9)
- moved R8 29.2 mm to (200.6, 178.2), turned to 180 degrees
- moved J11 28.8 mm to (203.9, 193.6)
- moved Q1 26.9 mm to (320.3, 203.0)
- moved R1 26.9 mm to (320.3, 193.1)
- moved JP1 26.0 mm to (306.2, 203.0), turned to 270 degrees
- moved J8 25.8 mm to (240.9, 99.5), turned to 180 degrees
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Connections:
- D3 pad 1: Fan+ -> 12V
- D3 pad 2: Fan- -> Controller-
- J1 pad 1: PFW -> 12V
- J1 pad 12: 12V -> PFW
- J1 pad 13: 5V_standby -> -12V
- J1 pad 24: -12V -> 5V_standby
- J10 pad 2: GND -> GND_HD
- J10 pad 3: GND -> GND_HD
- J11 pad 1: Fan- -> Controller-
- J11 pad 2: Fan+ -> 12V
- J12 pad 1: GND -> GND_HD
- J3 pad 2: GND -> GND_HD
- J3 pad 3: GND -> GND_HD
- J4 pad 2: GND -> GND_HD
- J4 pad 3: GND -> GND_HD
- J5 pad 2: GND -> GND_HD
- J5 pad 3: GND -> GND_HD
- J6 pad 2: GND -> GND_HD
- J6 pad 3: GND -> GND_HD
- J7 pad 2: GND -> GND_HD
- J7 pad 3: GND -> GND_HD
- J8 pad 2: GND -> GND_HD
- J8 pad 3: GND -> GND_HD
- J9 pad 2: GND -> GND_HD
- J9 pad 3: GND -> GND_HD
Routing:
- net 5V: track 761.2 -> 589.0 mm
- net 5V_HD: track 132.9 -> 226.0 mm
- net 5V_standby: track 205.9 -> 126.7 mm
- net 12V_HD: track 336.7 -> 285.0 mm
- net PFW: track 63.0 -> 13.6 mm
- net Fan+: track 40.7 -> 0.00 mm
- net Fan-: track 29.5 -> 0.00 mm
- net 12V: track 226.9 -> 207.0 mm
- net /LED_onoff: track 23.7 -> 6.06 mm
- net /-: track 15.7 -> 0.00 mm
- net PS_ON: track 70.0 -> 84.8 mm
- net Net-(C1-Pad1): track 6.27 -> 19.0 mm
- net Net-(D2-Pad2): track 22.0 -> 10.7 mm
- net /PWM_att: track 20.7 -> 10.6 mm
- net /PWM_signal: track 17.7 -> 27.7 mm
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- added copper zone on B.Cu, net GND_HD
Other:
- board text added: "DC v2.0"
- board text added: "ext. 12V Load Resistor"
- board text removed: "+12V"
- board text removed: "12V Load Resistors (only install if rail is unstable)"
- board text removed: "DC v1.02"
- board text removed: "From PSU"
- board text removed: "Monitor Relay"
- board text removed: "To Fan"
- board text removed: "w/ help from Geekdot, Stylurgys & Compgeke"
